File: badge.sch (EAGLE design)
At the start: 60 parts, among them J1 SJ-3523-SMT-TR, Q1 MMBT2222A-7-FSOT-23_DIO-M, Q2 MMBT2222A-7-FSOT-23_DIO-M, U1 MCP1703T-5002E, U2 SA602AD8-SOIC, U3 LM386M-1

Commit message: updates
* added ATTiny keyer and buttons
* added breakout jumper
* added images
* added README
Parts:
- added JP1: (no value), adafruit:PINHD-2X9-BIG
- added Q3: BSS138, Transistor:BSS138
- added R10, R11, R9: 10k, adafruit:R-US_M0805
- added R8: 4.7k, adafruit:R-US_M0805
- added SW1, SW2: 1825027-5, zort2:1825027-5
- added U4: ATTINY_402SOIC-8, zort2:ATTINY_402SOIC-8
Connections:
- removed net 6V_DC: C2.1, R2.1, U1.VO, U2.VCC
- removed net N$31: ANT.ANT, C30.1, L11.CA
- new net 5V_DC: C2.1, JP1.3, R10.1, R11.1, R2.1, R9.1, U1.VO, U2.VCC, U4.P$1
- new net ANT: ANT.ANT, C30.1, JP1.16, JP1.18, L11.CA
- new net AT2: JP1.7, U4.P$2
- new net AT3: JP1.9, R9.2, SW1.1, U4.P$3
- new net AT4: JP1.11, R10.2, SW2.1, U4.P$4
- new net AT5: JP1.13, Q3.G, R11.2, U4.P$5
- new net AT6: R8.1, U4.P$6
- new net AT7: JP1.17, U4.P$7
- new net N$42: JP1.8
- new net N$43: JP1.10
- new net N$44: JP1.12
- new net N$45: JP1.14
- new net PROGRAM: JP1.15, R8.2
- net GND: now also JP1.2, JP1.4, JP1.5, JP1.6, Q3.S, SW1.2, SW1.3, SW1.4, SW2.2, SW2.3, SW2.4, U4.P$8
- net HEADPHONE: now also J1.3
- net KEY_IN: now also Q3.D; no longer J1.3
- net VIN: now also JP1.1
Other:
- note added: "Keyer"
- note added: "Output Board"
- moved on the sheet: ANT

Commit message: moving to capacitive touch
Not ready for production

* replaced switches with capacitive touch buttons
* slight cleanup pass
Parts:
- removed SW1, SW2: 1825027-5, zort2:1825027-5
- added BTN1, BTN2: TOUCH_SMALL, zort2:TOUCH_SMALL
- added R12, R13, R14: 100, adafruit:R-US_M0805
- JP1: device adafruit:PINHD-2X9-BIG -> adafruit:PINHD-1X9
- R10, R9: value 10k -> 1M
Connections:
- net KEY_IN renamed Q1_GND
- removed net N$42: JP1.8
- removed net N$43: JP1.10
- removed net N$44: JP1.12
- removed net N$45: JP1.14
- new net KEY_SWITCH: JP1.3, Q3.G, R11.2, R14.2
- new net N$27: BTN1.P$1, R12.1, R9.2
- new net N$31: BTN2.P$1, R10.1, R13.2
- net 5V_DC: now also JP1.1; no longer JP1.3, R10.1, R11.1, R9.1
- net ANT: now also JP1.8, JP1.9; no longer JP1.16, JP1.18
- net AT2: now also R9.1; no longer JP1.7
- net AT3: now also R12.2; no longer JP1.9, R9.2, SW1.1
- net AT4: no longer JP1.11, SW2.1
- net AT5: now also R14.1; no longer JP1.13, Q3.G, R11.2
- net AT7: now also R13.1; no longer JP1.17
- net GND: now also BTN1.P$2, BTN2.P$2, JP1.7, R11.1; no longer JP1.2, SW1.2, SW1.3, SW1.4, SW2.2, SW2.3, SW2.4
- net PROGRAM: now also JP1.2; no longer JP1.15
- net VIN: no longer JP1.1
Other:
- moved on the sheet: Q3, R10, R11, R9
